Commit message: fix joints order

File: Section10_SLAM/bumperbot_ws/src/bumperbot_description/urdf/bumperbot_ros2_control.xacro (robot description, xacro)
@@ -25,5 +25,5 @@
         </xacro:unless>
         <!-- ros2_control Common Interfaces -->
-        <joint name="wheel_right_joint">
+        <joint name="wheel_left_joint">
             <command_interface name="velocity">
               <param name="min">-1</param>
@@ -33,5 +33,5 @@
             <state_interface name="velocity" />
         </joint>
-        <joint name="wheel_left_joint">
+        <joint name="wheel_right_joint">
             <command_interface name="velocity">
               <param name="min">-1</param>

File: Section11_Build_the_Robot/bumperbot_ws/src/bumperbot_description/urdf/bumperbot_ros2_control.xacro (robot description, xacro)
@@ -25,5 +25,5 @@
         </xacro:unless>
         <!-- ros2_control Common Interfaces -->
-        <joint name="wheel_right_joint">
+        <joint name="wheel_left_joint">
             <command_interface name="velocity">
               <param name="min">-1</param>
@@ -33,5 +33,5 @@
             <state_interface name="velocity" />
         </joint>
-        <joint name="wheel_left_joint">
+        <joint name="wheel_right_joint">
             <command_interface name="velocity">
               <param name="min">-1</param>
